File: hardware/interposer/rev0/rev0.kicad_sch (KiCad schematic)
At the start: 14 parts, among them J1 Z80_PLUG_TO_MB, J2 Z80_SOCKET_CPU, J3 5V_INPUT, U1 74AHCT165, U2 74AHCT165, U3 74AHCT165, U4 74AHCT165, U5 PICO_2_W

Commit message: docs: sweep the name to o1next, from the repository name downwards (#228)
One pass, because a half-renamed tree is worse than either name.  Paths move,
tokens change, and every generated artifact is regenerated from its source:

  o1nextgen  -> o1next       (2052 -> 0)
  o1ng       -> o1next       (  91 -> 0)
  O1NG       -> O1NEXT       ( 127 -> 0)
  osborne1ng -> osborne1nx   ( 184 -> 0, in the MAME context only)

Paths that move, content following:

  hardware/o1ng/                        -> hardware/o1next/
  hardware/o1ng/o1ng-lff/               -> hardware/o1next/o1next-lff/
  hardware/.../o1ng-lff.kicad_{pro,sch} -> o1next-lff.kicad_{pro,sch}
  docs/design/o1ng-lunchbox-concept.*   -> docs/design/o1next-lunchbox-concept.*
  research/boot-screen/o1ng-art.*       -> research/boot-screen/o1next-art-1ng.*
  site/hardware/o1ng-complete.md        -> site/hardware/o1next-complete.md
  site/assets/o1nextgen-logo.art.txt    -> site/assets/o1next-logo.art.txt
  site/assets/o1nextgen-logo.png        -> site/assets/o1next-logo.png
  site/assets/o1nextgen-wordmark.svg    -> site/assets/o1next-wordmark.svg
  docs/osborne1ng-machine.md            -> docs/osborne1nx-machine.md
  site/assets/osborne1ng-*.{mmd,png}    -> site/assets/osborne1nx-*.{mmd,png}
  tools/emulator-setup/mame-osborne1ng/ -> .../mame-osborne1nx/
  .../o1ng-{probe,dataphase}.lua        -> .../o1next-{probe,dataphase}.lua
  .../osborne1ng.patch                  -> .../osborne1nx.patch

The three site/assets paths, the two o1ng-lff.kicad_* files and the wordmark
were not in the issue's inventory; they were found by measuring the tree.

Generated, so regenerated rather than hand-edited:

  site/compendium/*, site/_includes/compendium-toc.html and the book PDF
    (tools/build_book.py -- its BLOB and front-matter author follow the name)
  site/assets/o1next-logo.png          (tools/research/rom2strokes.py --logo)
  research/boot-screen/o1next-frame.png (--frame --png)
  docs/fog-library{,-catalogue.tsv}: the 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
Other:
- title: o1nextgen interposer Rev 0 test probe -> o1next interposer Rev 0 test probe
Changed lines of the file:
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@@
 (kicad_sch (version 20230121) (generator "eeschema") (generator_version "7.0")
   (paper "A3")
-  (title_block (title "o1nextgen interposer Rev 0 test probe") (date "2026-10-10") (rev "0.1") (comment 1 "Snoop-only Z80 bus probe: pass-through socket, 4x 74AHCT165 PISO snapshot front end, Pico 2 W. NOT the production interposer."))
+  (title_block (title "o1next interposer Rev 0 test probe") (date "2026-10-10") (rev "0.1") (comment 1 "Snoop-only Z80 bus probe: pass-through socket, 4x 74AHCT165 PISO snapshot front end, Pico 2 W. NOT the production interposer."))
   (symbol (lib_id "local:Z80_DIP40") (at 59.69 90.17 0) (unit 1) (exclude_from_sim no) (in_bom yes) (on_board yes)
     (property "Reference" "J1" (at 59.69 34.29 0) (effects (font (size 1.27 1.27))))
