File: hardware/wifi-comm-pac/wifi-comm-pac.kicad_sch (KiCad schematic)
At the start: 71 parts, among them J1 Conn_02x05 IDC (P1 MODEM), J2 Speaker, J3 USB-C sink, SW1 Slide switch, latching, U1 74LVC4T245 (TXD/MCB 5V->3V3), U10 AP2112K-3.3 LDO, U2 74LVC4T245 (CTS/RI 3V3->5V), U3 74LVC1G07 (MSB open-drain), U4 MAX3232 (RXD bipolar), U5 ESP32-S2-MINI-2U, U6 AW9523B panel 0x58, U7 AW9523B interface 0x59, U8 MAX98357A, U9 TPS54331 buck 12.6->5

Commit message: hardware: wire the wifi-comm-pac nets instead of labelling them (#324 #325, part of #56) (#347)
The first sheet attached a net label to every pin and drew no wire between any two parts. It was electrically correct and read as a pile of disconnected stubs.

Now every signal net is drawn as orthogonal segments on a 1.27 mm grid, the rails use power symbols (with one PWR_FLAG per rail so ERC is satisfied), and exactly one label per net is kept so the net names survive - which also means a missing wire breaks the netlist instead of being hidden by a label. A Manhattan A* does the routing: symbol bodies impassable, another net's wire crossable but not runnable-along or endable-on, and another component's pin impassable - that last rule caught the first pass running wires through neighbouring pins, which shorted C2P to VP and C2N to C2P.

ERC is 0 errors; the 70-net netlist is unchanged, which is the check that the wires really do connect what the labels used to.
Parts:
- U1: value 74LVC4T245 (TXD/MCB 5V->3V3) -> 74LVC4T245 (TXD/MCB)
- U2: value 74LVC4T245 (CTS/RI 3V3->5V) -> 74LVC4T245 (CTS/RI)
- U3: value 74LVC1G07 (MSB open-drain) -> 74LVC1G07 (MSB)
- U4: value MAX3232 (RXD bipolar) -> MAX3232 (RXD)
Connections:
- net LED_MR_A: now also R10.2; no longer R10.1
- net LED_MR_K: now also R10.1; no longer R10.2
- net LED_RI_A: now also R11.2; no longer R11.1
- net LED_RI_K: now also R11.1; no longer R11.2
- net LED_TR_A: now also R9.2; no longer R9.1
- net LED_TR_K: now also R9.1; no longer R9.2
- no-connect marks 35 -> 27
Other:
- note added: "Power is diode-OR: 12.6 V -> 5 V path, and USB-C 5 V for bench work."
- note removed: "Audio is MAX98357A on +5V. Power is diode-OR: 12.6V path and USB-C path."
- note removed: "IC pin numbers here are LOGICAL; bind them at footprint annotation."

Commit message: hardware: the schematic gets its footprints, so it can become a board (#324 #325, part of #56)
`Update PCB from Schematic` transferred **nothing**, because all 200 Footprint
fields were empty.  That was deliberate -- the generator's own note said "the
real assignment is made at footprint annotation" -- and it is why the board
could not be started without hand-assigning 71 footprints in KiCad, which is the
hand transcription this generator exists to avoid.

**Every name added here was checked against KiCad's own libraries** before being
written down -- confirmed to exist as
`<kicad>/footprints/<lib>.pretty/<name>.kicad_mod`.  A footprint that does not
exist is worse than an empty one, because it *looks* assigned.

    footprints: 55 of 71 component symbols have one; 16 do not

The 14 filled types cover 55 instances: J1, U1/U2 (TSSOP-16), U3 (SOT-23-6),
U4 (SOIC-16), U6/U7 (QFN-24), U9 (SOIC-8), U10 (SOT-23-5), R x27, C x14, L,
D x3, F.  Keyed by SYMS key, so `R` is one line for 27 resistors.

**Seven types are left empty, and the generator names them on every run**,
because each is a part decision rather than a lookup -- and a plausible-but-wrong
footprint is a board that does not fit, which is worse than a blank one because a
blank one is visibly undone:

  U5  ESP32-S2-MINI-2U.  KiCad carries MINI-1 and -1U and NO -2U, and the -2
      series is a different pad layout, so this needs a footprint drawn from the
      Espressif datasheet -- a library lookup cannot supply it.
  U8  MAX98357A.  TQFN-16 3x3 mm or WLP; the ordering part number decides.
  J2  speaker connector -- no part chosen yet.
  J3  USB-C receptacle.  The symbol has 7 pins (VBUS, CC1, CC2, D+, D-, GND,
      SHIELD) and every 16P footprint has more pads than that, so assigning one
      here leaves pads unconnected on the board.  The symbol needs its doubled
      VBUS/GND pins added first.
  SW1 slide switch, latching -- no part chosen yet.
  LED 11 of them, at 3.5x2.8 mm.  KiCad carries only *vendo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
Parts:
- C1, C10, C11, C12, C13, C14, C2, C3, C4, C5, C6, C7, C8, C9: footprint (none) -> Capacitor_SMD:C_0603_1608Metric
- D12, D13, D14: footprint (none) -> Diode_SMD:D_SMA
- F1: footprint (none) -> Fuse:Fuse_1206_3216Metric
- J1: footprint (none) -> Connector_PinHeader_2.54mm:PinHeader_2x05_P2.54mm_Vertical
- L1: footprint (none) -> Inductor_SMD:L_1210_3225Metric
- R1, R10, R11, R12, R13, R14, R15, R16, R17, R18, R19, R2, R20, R21, R22, R23, R24, R25, R26, R27, R3, R4, R5, R6, R7, R8, R9: footprint (none) -> Resistor_SMD:R_0603_1608Metric
- U1, U2: footprint (none) -> Package_SO:TSSOP-16_4.4x5mm_P0.65mm
- U10: footprint (none) -> Package_TO_SOT_SMD:SOT-23-5
- U3: footprint (none) -> Package_TO_SOT_SMD:SOT-23-6
- U4: footprint (none) -> Package_SO:SOIC-16_3.9x9.9mm_P1.27mm
- U6, U7: footprint (none) -> Package_DFN_QFN:QFN-24-1EP_4x4mm_P0.5mm_EP2.6x2.6mm
- U9: footprint (none) -> Package_SO:SOIC-8_3.9x4.9mm_P1.27mm

Commit message: hardware: U8 is a TQFN-16, and five footprint decisions are now recorded (#324 #325, part of #56)
The six decisions from the issue, worked through.  One lands, five are now
*recorded* rather than open-ended -- each with what it needs, checked against the
actual source rather than assumed.

**Done: U8, the MAX98357A.**  `Package_DFN_QFN:TQFN-16-1EP_3x3mm_P0.5mm_EP1.6x1.6mm`.
The one variable is the exposed thermal pad: KiCad carries 1.6, 1.7 and 1.75 mm,
and neither analog.com nor farnell.com would serve a datasheet to this machine, so
1.6 is *chosen and said so* rather than checked.  It affects solderability, not
pin compatibility, and it is one word to change.

    footprints: 56 of 71 component symbols have one; 15 do not

**U5 is blocked, and it is not the library install.**  The Espressif KiCad library
carries ESP32-S2-MINI-1, -1U and SOLO-2U and **no MINI-2 or -2U** -- while MINI-1
and -1U are NRND, which is the whole reason pinmap.md chose the -2U.  And the land
patterns differ: the MINI-2U outline is 12.3 x 15.4 mm, so the -1U footprint is
not a substitute, and using it would be exactly the "close enough" this issue is
about.  Espressif publishes land-pattern source files and a .STEP model in
datasheet section 10.1, so it is drawable -- it is just not in the library.

**J3 is two changes, not one.**  The part is a 24-pin receptacle (A1-A12, B1-B12
plus shield) and the SYMBOL has 7 pins, so the symbol must be rebuilt with the
real pin map before a footprint means anything.  That touches the netlist, which
the checker asserts, so it is its own piece of work rather than a footnote.

**LED: the value is wrong as well as the footprint.**  SunLED XZM2CRK168WA is a
1.8 x 0.6 mm *right-angle* chip LED and the schematic calls it "3528".  The
nearest KiCad footprint is LED_Kingbright_APA1606_1.6x0.6mm_Horizontal -- a
different part.

**J2 and SW1** are recorded with what is known and what is not.  J2 is 2-pin THT
at 5.00 mm, but the Farnell datasheet would not download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
Parts:
- U8: footprint (none) -> Package_DFN_QFN:TQFN-16-1EP_3x3mm_P0.5mm_EP1.6x1.6mm

Commit message: hardware: six footprints land, and the board is one symbol rebuild from done (#324 #325, part of #56)
The SnapEDA models and the two dimensions settled it, and the whole set turned out
to be smaller than the last pass suggested:

    footprints: 70 of 71 component symbols have one; 1 does not
    70 components in the netlist, 70 with a footprint

**U8 -- the exposed pad is 1.1 x 1.1 mm**, read from the SnapEDA model for the
MAX98357AETE_T rather than guessed at.  That settles the 1.6/1.7/1.75 question and
means **KiCad's own library carries it after all**:
`Package_DFN_QFN:VQFN-16-1EP_3x3mm_P0.5mm_EP1.1x1.1mm`.  The previous commit had a
1.6 mm pad marked as *chosen*; it was wrong, and it is now checked.

**U5 -- the module.**  SnapEDA's `ESP32-S2-MINI-2U-N4`, and it cross-checks against
the datasheet: 0.85 mm pad pitch, rows at +/-7.0 mm, 0.8 x 0.4 mm pads.  It lives in
`footprints/o1next.pretty/` because Espressif's library has MINI-1/-1U and SOLO-2U
and no -2U -- so it is ours to give back, and the README says where.

**J2 is not a speaker, it is a piezo buzzer** -- Multicomp Pro MCKPT-G1340-3917,
12 Vp-p, 4 kHz, 80 dB, 9.5 nF.  Drawn at 5.08 mm pin pitch, which is the breadboard
measurement.  Worth knowing, because a piezo is driven differently from a coil
speaker and the symbol still calls it `CONN_SPK` / "Speaker".

**LED -- drawn from the dimensions**: two 0.8 mm square pads 1.8 mm apart on
centre, in a 1.8 x 0.6 x 1.5 mm right-angle package.  KiCad's nearest 1.6 x 0.6 mm
right-angle is a different part, which is the whole reason this one is ours.

**SW1** is SparkFun COM-10860, SPST 6.7 x 2.6 mm.  Their library is **CC BY 4.0**,
so the footprint is copied in *with attribution in its own descr* rather than
referenced -- referencing it made the ERC report
`footprint_link_issues: The current configuration does not include the footprint
library 'SparkFun-Switch'`, which the checker caught and which would also have
failed CI.  Copied, the board needs no external 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
Parts:
- D1, D10, D11, D2, D3, D4, D5, D6, D7, D8, D9: footprint (none) -> o1next:LED_SunLED_XZM2CRK168WA
- J2: footprint (none) -> o1next:Piezo_Buzzer_Multicomp_MCKPT-G1340-3917
- SW1: footprint (none) -> o1next:Slide_SPST_SMD_6.7x2.6mm
- U5: footprint (none) -> o1next:ESP32-S2-MINI-2U
- U8: footprint Package_DFN_QFN:TQFN-16-1EP_3x3mm_P0.5mm_EP1.6x1.6mm -> Package_DFN_QFN:VQFN-16-1EP_3x3mm_P0.5mm_EP1.1x1.1mm

Commit message: hardware: swap J2 to a real speaker, Same Sky CMS-151103-088SP (#325)
J2 was a piezo buzzer (Multicomp Pro MCKPT-G1340-3917). It is now a real
speaker, because the panel has to make the noise a modem makes -- dial tone,
DTMF, a ring cadence -- and neither an active buzzer (one note) nor a bare
piezo element (non-linear, thin across the band) can. The MAX98357A is an
I2S class-D amp with its own DAC, so the waveform is synthesised in firmware
and the transducer only has to be linear over 300-3400 Hz.

Part: Same Sky CMS-151103-088SP -- 15 x 11 x 3 mm rectangular frame, 0.7 W
(1.0 W max), 8 ohm, 90 dB at 0.7 W/10 cm, PEEK cone, Nd-Fe-B magnet,
solder-pad terminals, Fo 680-850 Hz in a 1 cc box. 8 ohm is the load the amp
wants. Pin 1 is the '+' terminal -- the datasheet gives the polarity, cone
forward on positive dc -- so pin 1 takes SPK_P.

The datasheet came from Same Sky directly, not Mouser: the Mouser link
returns an HTML interstitial, and sameskydevices.com hosts the PDF at
product/resource/<part>.pdf.

Symbol CONN_SPK renamed SPEAKER (it is the transducer, not a connector), and
the symbol's value is now the part number rather than the word "Speaker".
The piezo's footprint is deleted -- nothing uses it.

New: o1next:Speaker_SameSky_CMS-151103-088SP. The 15 x 11 mm body and the
courtyard are exact from the datasheet. The two solder pads are PLACED, NOT
READ: the mechanical drawing (page 2) is a figure, so pad size, spacing and
pad-to-edge offset do not extract as text. Drawn at 2.0 x 2.0 mm, 5.08 mm
apart, 0.3 mm proud of the frame edge. To be confirmed against the drawing.

That is a third category, and it gets its own name: FOOTPRINT_UNCONFIRMED.
FOOTPRINT_OPEN means no footprint and a part decision outstanding; this means
the footprint is assigned and the board is complete and opens, but a number
in it was placed rather than read. The generator prints both on every run.

Verified: generator runs clean, 70 of 71 component symbols have a footprint
(J3 alone is op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
Parts:
- removed J2: Speaker, o1next:Piezo_Buzzer_Multicomp_MCKPT-G1340-3917, symbol local:CONN_SPK
- added J2: CMS-151103-088SP, o1next:Speaker_SameSky_CMS-151103-088SP, symbol local:SPEAKER
Connections:
- net SPK_N: now also J2.2
- net SPK_P: now also J2.1
