File: hardware/floppy-adapter/floppy-adapter.kicad_sch (KiCad schematic)
At the start: 13 parts, among them J1 Conn_02x17 socket (O1 side), J2 Conn_02x17 header (OEM cable), J3 Conn_02x17 header (Gotek), J4 Gotek power, J5 Panel switch, Q1 AO3400A GND switch, U1 NC7SB3157P6X DS-A switch, U2 TPS22918 +5V switch

Commit message: hardware: the switch lead gets its series resistor, and the panel switch is documented (#62)
R5 (1k) is now in series in the panel-switch lead, and it should have been there in
the commit that introduced the lead: I wrote "a series resistor on that lead is Rev B
hardening" about a wire that leaves the board for the front panel, and then did not
fit it.  A part that costs nothing and answers a hazard the design had already
identified is not hardening, it is the design.

The lead now goes J5.2 -> R5 -> CTRL, with R1 on the control side, so the fail-safe
is unchanged: an unplugged lead is still a low, and a low is the physical drives.
1 k limits what a transient can push into three CMOS gates and a FET gate; the FET's
~630 pF gate turns in about a microsecond through it, which is irrelevant for a
switch a hand moves.  J5.2 is its own net now (`SW_LEAD`), asserted by name.

**The panel switch is documented as the maintainer described it**: a plain SPST flip
switch, **UP = the physical drives, DOWN = the Gotek**, and up is the fail-safe
position.  It is a series switch between the cable's +5 V and the control node, so
the two wires are interchangeable -- which is the reason the card-end connector is a
bare 2-pin 2.54 mm header expecting a Dupont housing.  The shrouded alternative
(JST PH 2.00 mm, the part the WiFi COMM PAC already uses for its keyboard-adapter
power port) is recorded with what it would buy (retention, no exposed 5 V pin) and
what it costs (PH housings and a crimp), as a one-footprint-line choice.

**And the two accepted cable-egress routes are written down** (sec.7, and the board
README): break the 34-pin run into parts that pass the pocket's ventilation slots
(Loxley's approach -- nothing on the machine is cut), or cut the case for a full-size
34-pin cable alongside the two switch wires.  The card is the same either way, which
is why J3 stays a full 2x17 header: the cable that arrives may be either, and unused
positions simply carry no wire.

Checked: `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
Parts:
- added R5: 1k (lead series), Resistor_THT:R_Axial_DIN0207_L6.3mm_D2.5mm_P7.62mm_Horizontal, symbol local:RES
Connections:
- net CTRL: now also R5.2; no longer J5.2
- new net SW_LEAD: J5.2, R5.1
Other:
- note added: "+5V (down) or leaves it to R1 (up), so up is the fail-safe position."
- note added: "PANEL SWITCH: UP = physical drives, DOWN = Gotek. It ties the lead to"
- note added: "R5 = 1k in series with the switch lead: it leaves the board, so it gets one."
- note removed: "De-energised = physical drives (fail-safe). J5 now carries microamps,"
- note removed: "not the 73 mA a relay coil wanted."
