File: hardware/wifi-comm-pac/wifi-comm-pac-edited/wifi-comm-pac.kicad_sch (KiCad schematic)
At the start: 71 parts, among them J1 Conn_02x05 IDC (P1 MODEM), J2 CMS-151103-088SP, J3 USB-C sink, SW1 Slide switch, latching, U1 74LVC4T245 (TXD/MCB), U10 AP2112K-3.3 LDO, U2 74LVC4T245 (CTS/RI), U3 74LVC1G07 (MSB), U4 MAX3232 (RXD), U5 ESP32-S2-MINI-2U, U6 AW9523B panel 0x58, U7 AW9523B interface 0x59, U8 MAX98357A, U9 TPS54331 buck 12.6->5

Commit message: hardware: bind U5 to the module's own 73 pads -- the 3V3-to-GND short is gone (#325)
U5's symbol had 18 pins numbered 1..18 against a footprint with 73 pads.  The
numbers collided by name while disagreeing in meaning: symbol pin 1 was +3V3 and
the module's pad 1 is GND1, so `Update PCB from Schematic` put 3.3 V on a ground
pad.  I asked which GPIO carried what; the answer was a lookup, and it was
written down in pinmap.md the whole time.

U5 now uses the part's own numbers, like J3, and all 73 pads are accounted for:

  pad  3     3V3           pad 45       EN
  pad  19    IO15 UART1 TX pad 20       IO16 O1 RXD
  pads 28,29 IO33,IO34 I2C
  pads 31-33 IO35,IO36,IO37 I2S
  pad  34    IO38 panel INTN     pad 25  IO21 interface INTN
  pads 23,24 IO19,IO20 USB D-/D+ (the only USB pins there are)
  33 ground pads -> GND          26 free GPIO + pad 27 -> no-connect

13 used + 33 ground + 27 unused = 73, which is exactly what the footprint has,
and the pin-versus-pad audit now reports U5 as a clean match.  **U5 has left
pin_partial**, which is the shape of the fix: a part leaves that list by using its
real pin numbers, not by being excused in it.

Three things made it work:

- **Stacked pins.**  The module has 33 ground pads and a symbol does not want 33
  GND pins.  `stack_onto()` hides 32 of them behind one visible pin, which is the
  vendor's own convention and why SnapEDA's 73-pad symbol is readable.  KiCad
  connects stacked pins, so the netlist carries all 33 numbers -- verified.
- **One power symbol per point, not per pin.**  With 33 pins at one coordinate the
  power loop drew 33 GND symbols on top of each other.  It now skips a coordinate
  it has already served.
- **The free GPIO are carried and marked no-connect, not omitted** -- 27 pads, so
  their pads are visibly unused instead of silently floating, and ERC has nothing
  to complain about rather than 27 pin_not_connected errors.

The pin map is the datasheet's, cross-checked against SnapEDA's symbol for the
pa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
Connections:
- net +3V3: now also U5.3 (3V3); no longer U5.1 (3V3)
- net ESP_EN: now also U5.45 (EN); no longer U5.3 (EN)
- net GND: now also U5.1 (GND), U5.30 (GND), U5.42 (GND), U5.43 (GND), U5.46 (GND), U5.47 (GND), U5.48 (GND), U5.49 (GND), U5.50 (GND), U5.51 (GND), U5.52 (GND), U5.53 (GND), U5.54 (GND), U5.55 (GND), U5.56 (GND), U5.57 (GND), U5.58 (GND), U5.59 (GND), U5.60 (GND), U5.61_1 (GND), U5.61_2 (GND), U5.61_3 (GND), U5.61_4 (GND), U5.61_5 (GND), U5.61_6 (GND), U5.61_7 (GND), U5.61_8 (GND), U5.61_9 (GND), U5.62 (GND), U5.63 (GND), U5.64 (GND), U5.65 (GND); no longer U5.18 (GND)
- net I2C_SCL: now also U5.29 (IO34); no longer U5.8 (IO34)
- net I2C_SDA: now also U5.28 (IO33); no longer U5.7 (IO33)
- net I2S_BCLK: now also U5.31 (IO35); no longer U5.9 (IO35)
- net I2S_DIN: now also U5.33 (IO37); no longer U5.11 (IO37)
- net I2S_LRCLK: now also U5.32 (IO36); no longer U5.10 (IO36)
- net INT_IF: now also U5.25 (IO21); no longer U5.13 (IO21)
- net INT_PANEL: now also U5.34 (IO38); no longer U5.12 (IO38)
- net O1_TXD_3V3: now also U5.20 (IO16); no longer U5.6 (IO16)
- net UART1_TX: now also U5.19 (IO15); no longer U5.5 (IO15)
- net USB_DM_ESP: now also U5.23 (IO19); no longer U5.14 (IO19)
- net USB_DP_ESP: now also U5.24 (IO20); no longer U5.15 (IO20)
- no-connect marks 37 -> 61

Commit message: hardware: free-GPIO header, keyed 5 V out with a current limit, ESD on USB-C in (#325)
Three additions, all of them before layout rather than after.

**J4 -- the 26 free GPIO, brought out to a 2x13 header.**  They were marked
no-connect, which is correct but *terminal*: the pad is on the module's footprint,
the header is not, and reaching it later means redoing the board.  2x13 exactly,
because that is the 26 GPIO and not 2x14 with grounds.

**It is left unpopulated and marked `dnp`**, so KiCad keeps it out of the BOM and
off the placement file -- the difference between "left unfitted on purpose" and
"we forgot to order it".  Pins are numbered the way a 2x13 is (odd row 1, even row
2) and named with the module's own IO names, so the silk says IO43 and that is
UART0 TXD without a datasheet:

  row 1: IO0 IO1 IO2 IO3 IO4 IO5 IO6 IO7 IO8 IO9 IO10 IO11 IO12
  row 2: IO13 IO14 IO17 IO18 IO26 IO39 IO40 IO41 IO42 IO43 IO44 IO45 IO46

One table in the generator builds U5's symbol, names the nets *and* labels the
header, and the checker asserts each of the 26 as an **exact pair** -- one U5 pad,
one J4 pin.  Three lists would drift, and the first thing to drift would be a pin
labelled IO18 that is really IO17, which is the worst bug possible on a header a
hobbyist is meant to use.  Verified from the netlist: 26 of 26 pins, odd/even
numbering, names matching the symbol.

**J5 -- 5 V out to the keyboard adapter, keyed.**  A JST PH side-entry SMD
(S2B-PH-SM4-TB, KiCad's own footprint, JST's own datasheet).  Fully shrouded with a
polarising slot, so the plug cannot go in the wrong way round and there is no
reverse-voltage case to design for.  Side entry, so the cable leaves parallel to
the board and straight out the front of the pocket.  2 A / 100 V / 2.0 mm pitch.

It hangs off the **diode-OR output**, so whichever source is present feeds it --
which is what lets the keyboard adapter drop its 12 V->5 V buck and keep only the
LDO.

**U11 -- the current limit on that port.**  D13/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
Parts:
- added D15: PESD5V0S1BA ESD, Diode_SMD:D_SOD-323, symbol local:D_ESD
- added J4: 2x13 header, GPIO breakout (DNP), Connector_PinHeader_2.54mm:PinHeader_2x13_P2.54mm_Vertical, symbol local:EXP_GPIO_2X13
- added J5: 5V out to keyboard adapter, Connector_JST:JST_PH_S2B-PH-SM4-TB_1x02-1MP_P2.00mm_Horizontal, symbol local:PWR_OUT_5V
- added R28: 27k, Resistor_SMD:R_0603_1608Metric, symbol local:R
- added U11: TPS2553 current limit ~0.95A, Package_TO_SOT_SMD:SOT-23-6, symbol local:TPS2553
Connections:
- net +5V: now also U11.1 (IN)
- net GND: now also D15.2, J5.2, R28.2, U11.2 (GND), U11.3 (/EN)
- net VBUS_IN: now also D15.1
- net IO6: now reaches U5.10 (IO6)
- net IO6: now also J4.13 (IO6)
- net IO7: now reaches U5.11 (IO7)
- net IO7: now also J4.15 (IO7)
- net IO8: now reaches U5.12 (IO8)
- net IO8: now also J4.17 (IO8)
- net IO9: now reaches U5.13 (IO9)
- net IO9: now also J4.19 (IO9)
- net IO10: now reaches U5.14 (IO10)
- net IO10: now also J4.21 (IO10)
- net IO11: now reaches U5.15 (IO11)
- net IO11: now also J4.23 (IO11)
- net IO12: now reaches U5.16 (IO12)
- net IO12: now also J4.25 (IO12)
- net IO13: now reaches U5.17 (IO13)
- net IO13: now also J4.2 (IO13)
- net IO14: now reaches U5.18 (IO14)
- net IO14: now also J4.4 (IO14)
- net IO17: now reaches U5.21 (IO17)
- net IO17: now also J4.6 (IO17)
- net IO18: now reaches U5.22 (IO18)
- net IO18: now also J4.8 (IO18)
- net IO26: now reaches U5.26 (IO26)
- net IO26: now also J4.10 (IO26)
- net IO39: now reaches U5.35 (IO39)
- net IO39: now also J4.12 (IO39)
- net IO40: now reaches U5.36 (IO40)
- net IO40: now also J4.14 (IO40)
- net IO41: now reaches U5.37 (IO41)
- net IO41: now also J4.16 (IO41)
- net IO42: now reaches U5.38 (IO42)
- net IO42: now also J4.18 (IO42)
- net IO43: now reaches U5.39 (IO43)
- net IO43: now also J4.20 (IO43)
- net IO0: now reaches U5.4 (IO0)
- net IO0: now also J4.1 (IO0)
- net IO44: now reaches U5.40 (IO44)
- net IO44: now also J4.22 (IO44)
- net IO45: now reaches U5.41 (IO45)
- net IO45: now also J4.24 (IO45)
- net IO46: now reaches U5.44 (IO46)
- net IO46: now also J4.26 (IO46)
- net IO1: now reaches U5.5 (IO1)
- net IO1: now also J4.3 (IO1)
- net IO2: now reaches U5.6 (IO2)
- net IO2: now also J4.5 (IO2)
- net IO3: now reaches U5.7 (IO3)
- net IO3: now also J4.7 (IO3)
- net IO4: now reaches U5.8 (IO4)
- net IO4: now also J4.9 (IO4)
- net IO5: now reaches U5.9 (IO5)
- net IO5: now also J4.11 (IO5)
- new net +5V_OUT: J5.1, U11.6 (OUT)
- new net ILIM_5V: R28.1, U11.5 (ILIM)
- no-connect marks 61 -> 36

Commit message: hardware: J1 is a right-angle shrouded IDC header, pin 1 on the left (#324)
This settles the board's one mechanical unknown, which the README has been
carrying as open item #1: the cable is keyed, but which end was pin 1 was not in
the schematic.

J1 was `PinHeader_2x05_P2.54mm_Vertical` -- a plain vertical pin header.  It is
now `IDC-Header_2x05_P2.54mm_Horizontal`: a DIN 41651 / IEC 60603-13 box header,
right angle and shrouded.  Two reasons and the second is the one that was wrong:

  1. the cable leaves the front of the floppy pocket, so it has to be right angle
  2. **the cable is keyed, and a keyed socket cannot go on plain pins.**  It needs
     the shroud with its polarising feature -- so the old footprint could not have
     accepted the cable it was chosen for

**Pin 1 on the left** falls out of the footprint's own geometry at rotation 0, and
that is worth writing down rather than leaving to whoever does layout: the pads
are at x=0 (odd) and x=2.54 (even) running in +Y, and the shroud body is offset +X
(4.38 to 13.28), so the mating face points +X.  Standing in front of it looking
in, your right hand is +Y and pin numbers increase with +Y -- so pin 1 is on the
left.  Checked against the footprint's actual coordinates, not assumed.

**The key is on the bottom, toward the PCB.**  The footprint has the rib inside
the shroud at y=7.13, between the third and fourth pin pairs.  Which way up the
part is fitted is a build instruction and not a schematic fact -- a footprint is
2D and has no "which way up" -- so it is recorded in pinmap.md and the symbol
comment rather than pretended into the netlist.

New `mech` field in check_schematics.py, because a footprint can be forced by the
*case* rather than by the circuit and no net assertion can see that.  Without it
the footprint could be swapped back to a plain vertical pin header and every check
would still pass.  Verified that it bites: reverting J1's footprint to the old one
produces the failure naming it.

Verified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
Parts:
- J1: footprint Connector_PinHeader_2.54mm:PinHeader_2x05_P2.54mm_Vertical -> Connector_IDC:IDC-Header_2x05_P2.54mm_Horizontal
